File: Radio/_autosave-Radio.kicad_pcb (KiCad board)
At the start: 2 copper layers, 17 parts, among them SW1 Bourns PEC11R, SW2 Bourns PEC11R, SW3 SW_Push, SW4 SW_Push, U1 LM386, U2 RDA5807M_Module

Commit message: Updated Schematic
Parts:
- added R3: 10K, Resistor_THT:R_Axial_DIN0204_L3.6mm_D1.6mm_P5.08mm_Horizontal, F.Cu at (169.6, 87.5)
- added R4: 10K, Resistor_THT:R_Axial_DIN0204_L3.6mm_D1.6mm_P5.08mm_Horizontal, F.Cu at (169.6, 84.3)
- added R5: 10K, Resistor_THT:R_Axial_DIN0204_L3.6mm_D1.6mm_P5.08mm_Horizontal, F.Cu at (169.6, 81.2)
- added R6: 10K, Resistor_THT:R_Axial_DIN0204_L3.6mm_D1.6mm_P5.08mm_Horizontal, F.Cu at (169.6, 78.0)
Connections:
- R1 pad 1: Net-(U1-+) -> Net-(U2-LOUT)
- SW1 pad A: Net-(A1-GPIO1) -> Net-(R3-Pad1)
- SW1 pad B: Net-(A1-GPIO2) -> Net-(R4-Pad1)
- SW2 pad A: Net-(A1-GPIO4) -> Net-(R5-Pad1)
- SW2 pad B: Net-(A1-GPIO5) -> Net-(R6-Pad1)
- U2 pad 8: Net-(U1-+) -> Net-(U2-LOUT)
